File: cruscotto/pcb/scheda-madre/s3-audio.kicad_sch (KiCad schematic)
At the start: 14 parts, among them J10 Verso P1 S3: 5V TXD RXD GND, J11 Verso P2 S3: IO19 IO11 IO12 I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, J12 Verso P6 Speak S3, K1 G2RL-2 DC5, K2 G2RL-2 DC5, Q9 AO3400A

Commit message: feat(pcb): D-059 wires soldered to the mainboard, re-routed; BOM with Farnell availability
- D-059: fan (J4), display NTC (J5) and S3 cables (J10-J12) on 26 AWG solder-wire pads instead of
  connectors; MicroSD, VAN and IMU modules soldered directly. Schematic sheets EL-002 rev B,
  EL-004 rev C, EL-005 rev B (27/10/2026); J11 moved 2.5 mm outward for J1 clearance.
- Placement and routing redone: 3987 tracks, 514 vias; DRC 0 errors, 0 unconnected, no hole or
  dangling warnings; 92 silkscreen warnings left.
- completa-sbroglio-scheda-madre.py: drill map so new vias keep the 0.25 mm hole-to-hole distance
  from every drill, including same-net ones.
- BOM: everything needed except consumables; parts shared with the Data Logger order flagged
  (LM2903B spare, EEEHB1C100R; second VAN and SD modules needed).
- tools/controlla-distinta-farnell.py (element14 Product Search API, key read from env or
  ~/.farnell_api_key, never printed) and the 27/10/2026 Farnell snapshot: 10 items not stocked
  (ESP32-WROOM-32E-H4, TPS54360B, LMR36510, LM74700-Q1, CH340C, AO3400A, SRR1260-8R2Y, HRO USB-C,
  7.3 mm tactile switches, AFB0412VA-00), 4 at zero stock.

Limits: routing checked only by DRC; nothing ordered, built or tested.

Co-Authored-By: Claude Opus 5.5 <noreply@anthropic.com>
Parts:
- J10, J11: footprint Connector_Molex:Molex_PicoBlade_53048-0410_1x04_P1.25mm_Horizontal -> Connector_Wire:SolderWire-0.127sqmm_1x04_P3.7mm_D0.48mm_OD1mm
- J12: footprint Connector_Molex:Molex_PicoBlade_53048-0210_1x02_P1.25mm_Horizontal -> Connector_Wire:SolderWire-0.127sqmm_1x02_P3.7mm_D0.48mm_OD1mm
Changed lines of the file:
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@@
 	(title_block
 		(title "Scheda madre cruscotto C3+AI - collegamento S3 e audio")
-		(date "2026-10-24")
-		(rev "A")
+		(date "2026-10-27")
+		(rev "B")
 		(company "Cruscotto C3+AI")
-		(comment 1 "C3AI-CR-EL-005 rev A - proposta preliminare, non verificata")
-		(comment 2 "D-028, D-029, D-039")
+		(comment 1 "C3AI-CR-EL-005 rev B - proposta preliminare, non verificata")
+		(comment 2 "D-028, D-029, D-039, D-059")
 		(comment 3 "Generato da tools/genera-schema-scheda-madre.py")
 	)
@@
 		(property "Reference" "J10" (at 60.96 73.66 0) (effects (font (size 1.27 1.27))))
 		(property "Value" "Verso P1 S3: 5V TXD RXD GND" (at 60.96 76.2 0) (effects (font (size 1.27 1.27))))
-		(property "Footprint" "Connector_Molex:Molex_PicoBlade_53048-0410_1x04_P1.25mm_Horizontal" (at 60.96 63.5 0) (hide yes) (effects (font (size 1.27 1.27))))
+		(property "Footprint" "Connector_Wire:SolderWire-0.127sqmm_1x04_P3.7mm_D0.48mm_OD1mm" (at 60.96 63.5 0) (hide yes) (effects (font (size 1.27 1.27))))
 		(property "Datasheet" "" (at 60.96 63.5 0) (hide yes) (effects (font (size 1.27 1.27))))
 		(property "Description" "P1 dal basso verso l’alto 5V, TXD, RXD, GND; UART0 della S3 non usata (riserva per la porta nascosta)" (at 60.96 63.5 0) (hide yes) (effects (font (size 1.27 1.27))))
@@
 		(property "Reference" "J11" (at 60.96 106.68 0) (effects (font (size 1.27 1.27))))
 		(property "Value" "Verso P2 S3: IO19 IO11 IO12 IO13" (at 60.96 109.22 0) (effects (font (size 1.27 1.27))))
-		(property "Footprint" "Connector_Molex:Molex_PicoBlade_53048-0410_1x04_P1.25mm_Horizontal" (at 60.96 96.52 0) (hide yes) (effects (font (size 1.27 1.27))))
+		(property "Footprint" "Connector_Wire:SolderWire-0.127sqmm_1x04_P3.7mm_D0.48mm_OD1mm" (at 60.96 96.52 0) (hide yes) (effects (font (size 1.27 1.27))))
 		(property "Datasheet" "" (at 60.96 96.52 0) (hide yes) (effects (font (size 1.27 1.27))))
 		(property "Description" "P2 da destra a sinistra IO19, IO11, IO12, IO13; P2 non porta massa: riferimento da J10 (P1)" (at 60.96 96.52 0) (hide yes) (effects (font (size 1.27 1.27))))
@@
 		(property "Reference" "J12" (at 63.5 125.73 0) (effects (font (size 1.27 1.27)) (justify left)))
 		(property "Value" "Verso P6 Speak S3" (at 63.5 128.27 0) (effects (font (size 1.27 1.27)) (justify left)))
-		(property "Footprint" "Connector_Molex:Molex_PicoBlade_53048-0210_1x02_P1.25mm_Horizontal" (at 60.96 127 0) (hide yes) (effects (font (size 1.27 1.27))))
+		(property "Footprint" "Connector_Wire:SolderWire-0.127sqmm_1x02_P3.7mm_D0.48mm_OD1mm" (at 60.96 127 0) (hide yes) (effects (font (size 1.27 1.27))))
 		(property "Datasheet" "" (at 60.96 127 0) (hide yes) (effects (font (size 1.27 1.27))))
 		(property "Description" "Uscita differenziale senza indicazione di polarità: nessun filo a massa, fase da verificare all’ascolto" (at 60.96 127 0) (hide yes) (effects (font (size 1.27 1.27))))

Commit message: feat(bom): S1/S2 Omron B3F-1050, Vishay NTCs with datasheet B value; LCSC cart cross-check
- S1/S2 = Omron B3F-1050 (6x6, 7.3 mm, 100 gf); RT1 = Vishay NTCS0805E3104FXT; display NTC = Vishay
  NTCLE100E3104JB0 (leaded). B value from the datasheets, to be used by the firmware (not B3950).
  Schematic EL-002/EL-005 values and board values updated; footprints unchanged, routing still valid
  (DRC 0 errors, 0 unconnected).
- BOM: LCSC cart of 28/10/2026 (86.37 USD + 13 USD shipping) covers most parts; Q1, L1, C3, R5, R38,
  fan, 22 uF 1206, 10k and 100k from other suppliers; prefer original Diodes AP2112K over the clone.

Co-Authored-By: Claude Opus 5.5 <noreply@anthropic.com>
Parts:
- S1, S2: value 6x6 H7,3 -> B3F-1050
Changed lines of the file:
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@@
 	(symbol (lib_id "Switch:SW_Push") (at 45.72 175.26 90) (unit 1) (exclude_from_sim no) (in_bom yes) (on_board yes) (dnp no)
 		(property "Reference" "S1" (at 49.53 173.99 90) (effects (font (size 1.27 1.27)) (justify right)))
-		(property "Value" "6x6 H7,3" (at 49.53 176.53 90) (effects (font (size 1.27 1.27)) (justify right)))
+		(property "Value" "B3F-1050" (at 49.53 176.53 90) (effects (font (size 1.27 1.27)) (justify right)))
 		(property "Footprint" "Button_Switch_THT:SW_PUSH_6mm_H7.3mm" (at 45.72 175.26 0) (hide yes) (effects (font (size 1.27 1.27))))
 		(property "Datasheet" "" (at 45.72 175.26 0) (hide yes) (effects (font (size 1.27 1.27))))
@@
 	(symbol (lib_id "Switch:SW_Push") (at 81.28 175.26 90) (unit 1) (exclude_from_sim no) (in_bom yes) (on_board yes) (dnp no)
 		(property "Reference" "S2" (at 85.09 173.99 90) (effects (font (size 1.27 1.27)) (justify right)))
-		(property "Value" "6x6 H7,3" (at 85.09 176.53 90) (effects (font (size 1.27 1.27)) (justify right)))
+		(property "Value" "B3F-1050" (at 85.09 176.53 90) (effects (font (size 1.27 1.27)) (justify right)))
 		(property "Footprint" "Button_Switch_THT:SW_PUSH_6mm_H7.3mm" (at 81.28 175.26 0) (hide yes) (effects (font (size 1.27 1.27))))
 		(property "Datasheet" "" (at 81.28 175.26 0) (hide yes) (effects (font (size 1.27 1.27))))
